File: electronics/Nutrient Management Control.brd (EAGLE design)
At the start: 87.3 x 71.1 mm, 28 parts, among them IC1 7407N, K1 SRM-1C-SL-5VDC, Q1 FQP30N06L, Q2 FQP30N06L, Q6 FDU3N40TU

Commit message: Just Microcontroller and control signals left todo
Parts:
- removed 24ACVS: (no value), Aeroponics Control:43650-0215
- added C2, C3: 100n, Aeroponics Control:C050-024X044
- added D10, D11, D12, D13, D14, D3, D4, D5, D7, D8, D9: 1N4004, Aeroponics Control:DO-41
- added DS4, DS5, ISEC: JST-XH-04-PIN-LONG-PAD, Aeroponics Control:JST-XH-04-PACKAGE-LONG-PAD
- added HEAT: (no value), Aeroponics Control:43650-0215
- added IC2, IC3: 7407N, Aeroponics Control:DIL14
- added K2: SRM-1C-SL-5VDC, Aeroponics Control:SRM1CSL5VDC
- added NP1, NP2, NP3, NP4, NP5, NP6, NP7, NP8, RORP, WV: JST-XH-02-PIN-LONG-PAD, Aeroponics Control:JST-XH-02-PACKAGE-LONG-PAD
- added Q10, Q11, Q12, Q13, Q3, Q4, Q5, Q7, Q8, Q9: FQP30N06L, Aeroponics Control:TO254P470X1016X2019-3P
- added Q14: FDU3N40TU, Aeroponics Control:TO229P250X658X985-3P
- added R10, R13, R15, R17, R19, R21, R23, R25, R27, R3, R7: 10k, Aeroponics Control:0204/7
- added R12, R14, R16, R18, R20, R22, R24, R26, R28, R4, R9: 1K, Aeroponics Control:0204/7
- added TDS2: JST-XH-03-PIN-LONG-PAD, Aeroponics Control:JST-XH-03-PACKAGE-LONG-PAD
- renumbered FM1 to TDS1, IPRSV to MIXP, IPUMP to UV, ISV to SUPP, PS1 to TS1
Connections:
- removed net +24VAC: 24ACVS.P$1, K1.5
- removed net -24VAC: 24ACVS.P$2, UV.P$1
- new net N$11: D4.A, NP3.2, Q4.2
- new net N$12: IC1.6, R7.1, R9.1
- new net N$14: Q4.1, R9.2
- new net N$15: D5.A, NP5.2, Q5.2
- new net N$16: IC1.10, R10.1, R12.1
- new net N$18: Q5.1, R12.2
- new net N$19: D7.A, NP7.2, Q7.2
- new net N$2: D3.A, NP1.2, Q3.2
- new net N$20: IC2.2, R13.1, R14.1
- new net N$22: Q7.1, R14.2
- new net N$23: D8.A, NP2.2, Q8.2
- new net N$24: IC1.4, R15.1, R16.1
- new net N$25: Q8.1, R16.2
- new net N$26: D9.A, NP4.2, Q9.2
- new net N$27: IC1.8, R17.1, R18.1
- new net N$28: Q9.1, R18.2
- new net N$29: D10.A, NP6.2, Q10.2
- new net N$30: IC1.12, R19.1, R20.1
- new net N$31: Q10.1, R20.2
- new net N$32: D11.A, NP8.2, Q11.2
- new net N$33: IC2.4, R21.1, R22.1
- new net N$34: Q11.1, R22.2
- new net N$35: D12.A, Q12.2, RORP.2
- new net N$36: IC2.10, R23.1, R24.1
- new net N$37: Q12.1, R24.2
- new net N$38: D13.A, Q13.2, WV.2
- new net N$39: IC2.12, R25.1, R26.1
- new net N$40: Q13.1, R26.2
- new net N$41: D14.A, K2.1, Q14.2
- new net N$42: HEAT.P$2, K2.3
- new net N$43: Q14.1, R28.2
- new net N$44: IC3.4, R27.1, R28.1
- new net N$47: DS4.3
- new net N$48: DS4.4
- new net N$49: DS5.3
- new net N$50: DS5.4
- new net N$6: IC1.2, R3.1, R4.1
- new net N$8: Q3.1, R4.2
- net +12V: now also D10.C, D11.C, D12.C, D13.C, D3.C, D4.C, D5.C, D7.C, D8.C, D9.C, NP1.1, NP2.1, NP3.1, NP4.1, NP5.1, NP6.1, NP7.1, NP8.1, R27.2, RORP.1, WV.1
- net +240VAC: now also K1.5, K2.5
- net +5V: now also C2.1, C3.1, D14.C, DS4.1, DS5.1, IC2.14, IC3.14, K2.4, R10.2, R13.2, R15.2, R17.2, R19.2, R21.2, R23.2, R25.2, R3.2, R7.2, TDS2.1
- net -240VAC: now also HEAT.P$1, UV.P$1
- net DS1RX: no longer DS1.3
- net DS1TX: no longer DS1.4
- net DS2RX: no longer DS2.3
- net DS2TX: no longer DS2.4
- net DS3RX: no longer DS3.3
- net DS3TX: no longer DS3.4
- net FM1S: no longer TDS1.3
- net GND: now also C2.2, C3.2, DS4.2, DS5.2, IC2.7, IC3.7, Q10.3, Q11.3, Q12.3, Q13.3, Q14.3, Q3.3, Q4.3, Q5.3, Q7.3, Q8.3, Q9.3, TDS2.2
- net IPCTL: no longer IC1.11
- net IPRSVCTL: no longer IC1.3
- net ISVCTL: no longer IC1.1
- net N$17: now also IC3.2; no longer IC1.10
- net N$3: now also IC2.8; no longer IC1.2
- net N$9: now also IC2.6; no longer IC1.4
- net PS1S: no longer TS1.3
Routing:
- net N$17: track 20.2 -> 146.7 mm
- net N$9: track 66.9 -> 137.5 mm
- net N$3: track 49.4 -> 113.8 mm
- net -24VAC: track 21.1 -> 0.00 mm
- net +24VAC: track 13.4 -> 0.00 mm
- net IPRSVCTL: track 43.9 -> 35.3 mm
- net FM1S: track 38.0 -> 35.3 mm
- net DS2RX: track 61.9 -> 59.2 mm
- net DS1RX: track 38.5 -> 37.2 mm

Commit message: First cut of Nutrient Management electronics
Parts:
- removed PCB1: ARDUINO_NANOARDUINO_NANO_HEADERS, Aeroponics Control:ARDUINO_NANO
- added PCB2: ARDUINO_MEGA2560_SHIELD, Aeroponics Control:ARDUINO_MEGA2560_SHIELD
- renumbered NP7 to PHDPP, NP8 to PHUPP
Connections:
- removed net 5V: PCB1.12
- removed net DS1RX: PCB1.20
- removed net DS1TX: PCB1.21
- removed net DS2RX: PCB1.22
- removed net DS2TX: PCB1.23
- removed net DS3RX: PCB1.9
- removed net DS3TX: PCB1.8
- removed net FM1S: PCB1.4
- removed net IPCTL: PCB1.30
- removed net IPRSVCTL: PCB1.25
- removed net ISVCTL: PCB1.24
- removed net N$47: DS4.3
- removed net N$48: DS4.4
- removed net N$49: DS5.3
- removed net N$50: DS5.4
- removed net PS1S: PCB1.11
- removed net TP1CTL: PCB1.26
- removed net TP2CTL: PCB1.27
- removed net UVLCTL: PCB1.29
- new net HEATCTL: IC3.3, PCB2.32
- new net MIXPCTL: IC2.5, PCB2.2
- new net MTDO: DS1.4, PCB2.23
- new net MTT: PCB2.22, TS1.3
- new net N1PP: IC1.1, PCB2.34
- new net N2PP: IC1.3, PCB2.36
- new net N3PP: IC1.5, PCB2.38
- new net N4PP: IC1.9, PCB2.40
- new net N5PP: IC1.11, PCB2.42
- new net N6PP: IC1.13, PCB2.44
- new net PHDPP: IC2.1, PCB2.46
- new net PHUPP: IC2.3, PCB2.48
- new net RORPCTL: IC2.11, PCB2.4
- new net RRTDO: DS3.4, PCB2.27
- new net STDO: DS2.4, PCB2.25
- new net SUPPCTL: IC2.9, PCB2.3
- new net SWTDO: DS5.4, PCB2.31
- new net TDS1: PCB2.24, TDS1.3
- new net TDS2: PCB2.26, TDS2.3
- new net UVCTL: IC3.1, PCB2.30
- new net WVCTL: IC2.13, PCB2.49
- new net WWTDO: DS4.4, PCB2.29
- net +5V: now also DS1.3, DS2.3, DS3.3, DS4.3, DS5.3, PCB2.AREF, PCB2.VIN; no longer PCB1.15, PCB1.3
- net GND: now also IC3.10, IC3.11, IC3.12, IC3.13, IC3.5, IC3.6, IC3.8, IC3.9, PCB2.GND; no longer PCB1.14, PCB1.19
Routing:
- net +5V: track 254.3 -> 0.00 mm
- net GND: track 226.6 -> 0.00 mm, vias 1 -> 0
- net +12V: track 170.4 -> 0.00 mm, vias 1 -> 0
- net N$17: track 146.7 -> 0.00 mm
- net N$9: track 137.5 -> 0.00 mm
- net N$3: track 113.8 -> 0.00 mm
- net IPCTL: track 60.9 -> 0.00 mm
- net DS2RX: track 59.2 -> 0.00 mm
- net N$21: track 55.4 -> 0.00 mm
- net DS2TX: track 55.1 -> 0.00 mm, vias 1 -> 0
- net UVLCTL: track 51.2 -> 0.00 mm, vias 2 -> 0
- net -240VAC: track 47.1 -> 0.00 mm
- net TP1CTL: track 44.6 -> 0.00 mm
- net N$13: track 43.6 -> 0.00 mm
- net DS3RX: track 43.5 -> 0.00 mm
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
Commit message: First cut of Nutrient Management with multi UART breakout boards
Parts:
- removed DS1, DS2, DS3, DS4, DS5: JST-XH-04-PIN-LONG-PAD, Aeroponics Control:JST-XH-04-PACKAGE-LONG-PAD
- added MTDS, RRTDS, STDS, SWTDS, WWTDS: JST-XH-04-PIN-LONG-PAD, Aeroponics Control:JST-XH-04-PACKAGE-LONG-PAD
- moved PCB2 503.8 mm to (-10.2, 14.0)
- moved C3 480.1 mm to (22.9, 48.3), turned to 90 degrees
- moved C2 450.9 mm to (22.9, 36.8), turned to 90 degrees
- moved ISEC 443.5 mm to (97.8, 40.6), turned to 90 degrees
- moved HEAT 409.6 mm to (99.1, 53.3), turned to 270 degrees
- moved TDS2 403.7 mm to (97.8, 26.7), turned to 90 degrees
- moved D14 382.6 mm to (34.3, 30.5), turned to 90 degrees
- moved Q13 382.0 mm to (72.4, 69.8), turned to 180 degrees
- moved R27 380.0 mm to (31.8, 21.6)
- moved R28 380.0 mm to (41.9, 21.6)
- moved R25 374.1 mm to (90.2, 50.8), turned to 90 degrees
- moved Q14 373.4 mm to (25.4, 11.4)
- moved D13 370.9 mm to (94.0, 53.3), turned to 90 degrees
- moved K2 362.5 mm to (64.8, 26.7)
- moved R26 352.5 mm to (91.4, 30.5), turned to 90 degrees
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Connections:
- net +5V: now also MTDS.1, MTDS.3, RRTDS.1, RRTDS.3, STDS.1, STDS.3, SWTDS.1, SWTDS.3, WWTDS.1, WWTDS.3; no longer DS1.1, DS1.3, DS2.1, DS2.3, DS3.1, DS3.3, DS4.1, DS4.3, DS5.1, DS5.3
- net GND: now also MTDS.2, RRTDS.2, STDS.2, SWTDS.2, WWTDS.2; no longer DS1.2, DS2.2, DS3.2, DS4.2, DS5.2
- net MTDO: now also MTDS.4; no longer DS1.4
- net RRTDO: now also RRTDS.4; no longer DS3.4
- net STDO: now also STDS.4; no longer DS2.4
- net SWTDO: now also SWTDS.4; no longer DS5.4
- net WWTDO: now also WWTDS.4; no longer DS4.4
Routing:
- net +5V: track 0.00 -> 457.6 mm, vias 0 -> 7
- net GND: track 0.00 -> 434.2 mm, vias 0 -> 2
- net N$35: track 0.00 -> 262.7 mm, vias 0 -> 1
- net +12V: track 0.00 -> 251.7 mm, vias 0 -> 1
- net N5PP: track 0.00 -> 154.9 mm, vias 0 -> 2
- net N$39: track 0.00 -> 150.7 mm, vias 0 -> 3
- net N$21: track 0.00 -> 147.3 mm, vias 0 -> 2
- net N$29: track 0.00 -> 144.3 mm, vias 0 -> 5
- net WWTDO: track 0.00 -> 131.9 mm, vias 0 -> 3
- net N$19: track 0.00 -> 131.4 mm, vias 0 -> 5
- net N$26: track 0.00 -> 131.3 mm, vias 0 -> 7
- net N$14: track 0.00 -> 128.6 mm, vias 0 -> 3
- net N$1: track 0.00 -> 127.7 mm, vias 0 -> 4
- net PHUPP: track 0.00 -> 126.5 mm, vias 0 -> 4
- net N$20: track 0.00 -> 125.4 mm, vias 0 -> 6
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Other:
- board size 87.3 x 71.1 mm -> 101.6 x 81.3 mm
- board text removed: "24VAC"
- board text removed: "IPUMP"
